Commit message: 深度相机D435的插入与调试

File: cyberdog_sim/src/cyberdog_simulator/cyberdog_robot/cyberdog_description/xacro/gazebo.xacro (robot description, xacro)
@@ -98,4 +98,59 @@
         </gazebo>
     </xacro:if>
+    <!-- D435 Camera，仿照 RGB 相机方式挂载在 D435 预留安装位 -->
+    <xacro:if value="$(arg USE_D435_CAMERA)">
+        <gazebo reference="D435_camera_link">
+            <sensor name="d435_camera_sensor" type="camera">
+                <always_on>true</always_on>
+                <update_rate>30</update_rate>
+                <visualize>true</visualize>
+                <pose>0 0 0 0 0 0</pose>
+                <camera>
+                    <horizontal_fov>1.3962634</horizontal_fov>
+                    <image>
+                        <width>640</width>
+                        <height>480</height>
+                        <format>R8G8B8</format>
+                    </image>
+                    <clip>
+                        <near>0.05</near>
+                        <far>30.0</far>
+                    </clip>
+                </camera>
+                <plugin name="d435_camera_plugin" filename="libgazebo_ros_camera.so">
+                    <ros>
+                        <remapping>~/image_raw:=d435/color/image_raw</remapping>
+                        <remapping>~/camera_info:=d435/color/camera_info</remapping>
+                    </ros>
+                    <frame_name>D435_camera_link</frame_name>
+                </plugin>
+            </sensor>
+            <sensor name="d435_depth_sensor" type="depth">
+                <always_on>true</always_on>
+                <update_rate>30</update_rate>
+                <visualize>true</visualize>
+                <pose>0 0 0 0 0 0</pose>
+                <camera>
+                    <horizontal_fov>1.3962634</horizontal_fov>
+                    <image>
+                        <width>640</width>
+                        <height>480</height>
+                        <format>R8G8B8</format>
+                    </image>
+                    <clip>
+                        <near>0.05</near>
+                        <far>30.0</far>
+                    </clip>
+                </camera>
+                <plugin name="d435_depth_plugin" filename="libgazebo_ros_camera.so">
+                    <ros>
+                        <remapping>~/image_raw:=d435/depth/image_raw</remapping>
+                        <remapping>~/camera_info:=d435/depth/camera_info</remapping>
+                    </ros>
+                    <frame_name>D435_camera_link</frame_name>
+                </plugin>
+            </sensor>
+        </gazebo>
+    </xacro:if>
     <!-- Foot contacts. -->
     <gazebo reference="FR_knee">

File: cyberdog_sim/src/cyberdog_simulator/cyberdog_robot/cyberdog_description/xacro/robot.xacro (robot description, xacro)
@@ -9,4 +9,5 @@
     <xacro:arg name="USE_LIDAR" default="false" />
     <xacro:arg name="USE_RGB_CAMERA" default="false" />
+    <xacro:arg name="USE_D435_CAMERA" default="false" />
     <!-- 引入常量、腿部宏和 Gazebo 扩展配置 -->
     <xacro:include filename="const.xacro" />
@@ -89,5 +90,5 @@
         <parent link="body" />
         <child link="D435_camera_link" />
-        <origin rpy="0 0 0" xyz="271.994e-3 25e-3 114.912e-3" />
+        <origin rpy="0 1.00 0" xyz="271.994e-3 25e-3 114.912e-3" />
     </joint>
     <link name="D435_camera_link">
