Commit message: yxy_1

File: cyberdog_sim/src/cyberdog_simulator/cyberdog_robot/cyberdog_description/xacro/robot.xacro (robot description, xacro)
@@ -9,5 +9,4 @@
     <xacro:arg name="USE_LIDAR" default="false" />
     <xacro:arg name="USE_RGB_CAMERA" default="false" />
-    <xacro:arg name="USE_D435_CAMERA" default="false" />
     <!-- 引入常量、腿部宏和 Gazebo 扩展配置 -->
     <xacro:include filename="const.xacro" />
@@ -90,5 +89,5 @@
         <parent link="body" />
         <child link="D435_camera_link" />
-        <origin rpy="0 1.00 0" xyz="271.994e-3 25e-3 114.912e-3" />
+        <origin rpy="0 0 0" xyz="271.994e-3 25e-3 114.912e-3" />
     </joint>
     <link name="D435_camera_link">

Commit message: 二维码的识别与扫描

File: cyberdog_sim/src/cyberdog_simulator/cyberdog_robot/cyberdog_description/xacro/robot.xacro (robot description, xacro)
@@ -89,5 +89,5 @@
         <parent link="body" />
         <child link="D435_camera_link" />
-        <origin rpy="0 0 0" xyz="271.994e-3 25e-3 114.912e-3" />
+        <origin rpy="0 1 0" xyz="271.994e-3 25e-3 114.912e-3" />
     </joint>
     <link name="D435_camera_link">
